File: rpi-q5-adapter/rpi-q5-adapter.kicad_pcb (KiCad board)
At the start: 2 copper layers, 51.1 x 54.3 mm, 46 parts, among them J1 Conn_01x15, J2 Conn_02x15_Odd_Even, J3 Raspberry_Pi_2_3, Q1 BC847, U1 SGM2019-2.8YN5G/TR, U2 SGM2019-1.8YN5G/TR, U3 PCA9536D, U4 SGM3204YN6G/TR, U5 CAT4139

Commit message: mipi trace tuning
Parts:
- D1: value D_Zener -> D_Schottky
- D2: value DIODE -> type="D" model="DIODE" lib=""
- renumbered TP5 to -5V1, TP3 to 1V8, TP2 to 2V8, TP1 to 3V3, TP4 to 5V1, TP6 to BL_A1, TP7 to BL_K1
Routing:
- net /D1_N: track 19.8 -> 24.9 mm
- net /D1_P: track 20.5 -> 25.7 mm
- net /RESET: track 64.5 -> 62.4 mm
- net /D0_P: track 24.3 -> 25.8 mm
- net /D0_N: track 23.6 -> 25.1 mm
- net /LCD_A: track 28.7 -> 28.1 mm
- net GND: vias 272 -> 286
