File: rpi-q5-adapter/rpi-q5-adapter.kicad_sch (KiCad schematic)
At the start: 46 parts, among them J1 Conn_01x15, J2 Conn_02x15_Odd_Even, J3 Raspberry_Pi_2_3, Q1 BC847, U1 SGM2019-2.8YN5G/TR, U2 SGM2019-1.8YN5G/TR, U3 PCA9536D, U4 SGM3204YN6G/TR, U5 CAT4139

Commit message: mipi trace tuning
Parts:
- D2: value DIODE -> ${SIM.PARAMS}; Spice_Netlist_Enabled Y -> (none); Spice_Primitive D -> (none)
- renumbered TP5 to -5V1, TP3 to 1V8, TP2 to 2V8, TP1 to 3V3, TP4 to 5V1, TP6 to BL_A1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
